File: PCB Related/PiHome Temp Sensors/PiHome Temp Sensors.brd (EAGLE design)
At the start: 71.1 x 50.8 mm, 12 parts, among them M1 WIRELESS-NRF24L01, U1 DS18B20

Commit message: openhardware logo
open hardware logo added
Parts:
- added LOGO1: OSHW-LOGOL, SparkFun-Aesthetics:OSHW-LOGO-L
Changed lines of the file:
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@@
 </element>
 <element name="U$1" library="Arduino Pro Mini-Nano" package="ABK-PRO-MINI" value="ABK-PRO-MINI" x="57.785" y="36.83" rot="R270"/>
+<element name="LOGO1" library="SparkFun-Aesthetics" package="OSHW-LOGO-L" value="OSHW-LOGOL" x="14.605" y="38.735"/>
 </elements>
 <signals>
