File: PCB Related/PiHome Temp Sensors/PiHome Temp Sensors.brd (EAGLE design)
At the start: 71.1 x 50.8 mm, 13 parts, among them M1 WIRELESS-NRF24L01, U1 DS18B20

Commit message: PiHome – Smart Heating Controller
PCB improvements
Parts:
- moved BAT1 0.63 mm to (35.6, 12.7)
Changed lines of the file:
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@@
 <?xml version="1.0" encoding="utf-8"?>
 <!DOCTYPE eagle SYSTEM "eagle.dtd">
-<eagle version="7.5.0">
+<eagle version="9.0.1">
 <drawing>
 <settings>
 <setting alwaysvectorfont="no"/>
+<setting keepoldvectorfont="yes"/>
 <setting verticaltext="up"/>
 </settings>
@@
 <layer number="45" name="Holes" color="7" fill="1" visible="yes" active="yes"/>
 <layer number="46" name="Milling" color="3" fill="1" visible="no" active="yes"/>
-<layer number="47" name="Measures" color="7" fill="1" visible="no" active="yes"/>
+<layer number="47" name="Measures" color="7" fill="1" visible="yes" active="yes"/>
 <layer number="48" name="Document" color="7" fill="1" visible="yes" active="yes"/>
 <layer number="49" name="Reference" color="7" fill="1" visible="yes" active="yes"/>
@@
 <text x="37.7825" y="48.26" size="0.8128" layer="21" ratio="10">VCC</text>
 <hole x="3.81" y="46.99" drill="3.81"/>
-<hole x="3.81" y="3.81" drill="3.81"/>
-<hole x="68.58" y="3.81" drill="3.81"/>
-<hole x="68.58" y="46.99" drill="3.81"/>
+<hole x="3.81" y="4.7625" drill="3.81"/>
+<hole x="66.04" y="4.7625" drill="3.81"/>
+<hole x="66.04" y="47.3075" drill="3.81"/>
 <text x="53.975" y="1.27" size="1.016" layer="21">Rev:1 - Sketch 1.34</text>
 <hole x="67.31" y="19.685" drill="0.6"/>
 <text x="51.435" y="48.895" size="0.8128" layer="21" ratio="10">Off</text>
 <text x="57.15" y="48.895" size="0.8128" layer="21" ratio="10">On</text>
+<dimension x1="0" y1="50.8" x2="71.12" y2="50.8" x3="35.56" y3="59.69" textsize="1.778" layer="47"/>
+<dimension x1="3.81" y1="46.99" x2="66.04" y2="46.99" x3="34.925" y3="53.34" textsize="1.778" layer="47"/>
+<dimension x1="3.81" y1="46.99" x2="3.81" y2="4.7625" x3="-1.905" y3="25.87625" textsize="1.778" layer="47"/>
+<dimension x1="0" y1="0" x2="0" y2="50.8" x3="-6.35" y3="25.4" textsize="1.778" layer="47"/>
+<dimension x1="3.81" y1="4.7625" x2="66.04" y2="4.7625" x3="34.925" y3="-1.905" textsize="1.778" layer="47"/>
+<dimension x1="66.04" y1="4.7625" x2="66.04" y2="46.99" x3="74.295" y3="25.87625" textsize="1.778" layer="47"/>
 </plain>
 <attributes>
@@
 <param name="dpMaxLengthDifference" value="10mm"/>
 <param name="dpGapFactor" value="2.5"/>
-<param name="checkGrid" value="0"/>
 <param name="checkAngle" value="0"/>
 <param name="checkFont" value="1"/>
 <param name="checkRestrict" value="1"/>
+<param name="checkStop" value="0"/>
+<param name="checkValues" value="0"/>
 <param name="useDiameter" value="13"/>
 <param name="maxErrors" value="50"/>
@@
 </autorouter>
 <elements>
-<element name="BAT1" library="SparkFun-Electromechanical" package="BATTERY_18650-HOLDER" value="" x="35.56" y="12.065" smashed="yes" rot="R180">
-<attribute name="VALUE" x="63.5" y="13.335" size="0.4064" layer="27" rot="R180"/>
+<element name="BAT1" library="SparkFun-Electromechanical" package="BATTERY_18650-HOLDER" value="" x="35.56" y="12.7" smashed="yes" rot="R180">
+<attribute name="VALUE" x="63.5" y="13.97" size="0.4064" layer="27" rot="R180"/>
 </element>
 <element name="C1" library="SparkFun-Capacitors" package="CAP-PTH-SMALL-KIT" value="0.1uf" x="29.21" y="28.575" rot="R180">
@@
 <via x="67.31" y="19.685" extent="1-16" drill="0.6"/>
 <wire x1="67.31" y1="19.685" x2="67.31" y2="13.197" width="0.4064" layer="16"/>
-<wire x1="67.31" y1="13.197" x2="66.188" y2="12.075" width="0.4064" layer="16"/>
+<wire x1="67.31" y1="13.197" x2="66.188" y2="12.71" width="0.4064" layer="16"/>
 </signal>
 <signal name="TXO">

Commit message: Improved PCB Design
Improved PCB Design
Parts:
- added LED1: (no value), adafruit:LED3MM
- added R5: 220Ohm, SparkFun-Resistors:AXIAL-0.3
- moved U1 2.84 mm to (4.45, 25.4)
- moved LOGO1 2.62 mm to (14.0, 41.3)
- moved M1 1.27 mm to (17.8, 38.7)
- moved R1 1.27 mm to (56.5, 31.8)
- moved R2 1.27 mm to (54.6, 34.3)
- moved BAT1 1.27 mm to (35.6, 11.4)
- moved C3 1.27 mm to (29.2, 22.9)
- moved R3 1.27 mm to (17.8, 27.9)
- moved C2 1.27 mm to (47.6, 33.0)
- moved JP1 1.27 mm to (40.0, 45.1)
- moved S1 1.27 mm to (54.6, 45.1)
- moved U$1 1.27 mm to (57.8, 35.6)
- moved C1 0.63 mm to (29.2, 27.9), turned to 0 degrees
Connections:
- new net D4: R5.P$1, U$1.D4
- new net N$1: LED1.A, R5.P$2
- net GND: now also LED1.K
Routing:
- net D4: track 0.00 -> 38.4 mm, vias 0 -> 1
- net N$1: track 0.00 -> 8.45 mm, vias 1 -> 0
- net SCK: track 37.1 -> 29.7 mm
- net MOSI: track 26.0 -> 19.9 mm
- net VDD: track 56.7 -> 60.7 mm
- net 3.3V: track 66.0 -> 69.1 mm
- net CSN: track 14.3 -> 16.3 mm
- net VCC: track 27.7 -> 25.9 mm
- net MISO: track 21.1 -> 22.4 mm
- net RXI: track 34.7 -> 34.0 mm
Other:
- board size 71.1 x 50.8 mm -> 70.5 x 48.3 mm
- board text added: "DS18B20"
- board text added: "PiHome - Smart Heating"
- board text added: "Temperature Sensor"
- board text added: "nRF24L01 / 2.4GHz"
- board text removed: "PiHome Temperature Sensor"
- board text removed: "nRF24L01 / 2.4GHz RF"
