File: PCB Related/PiHome Temp Sensors/PiHome Temp Sensors.sch (EAGLE design)
At the start: 12 parts, among them M1 WIRELESS-NRF24L01, U1 DS18B20

Commit message: openhardware logo
open hardware logo added
Parts:
- added LOGO1: OSHW-LOGOL, SparkFun-Aesthetics:OSHW-LOGOL
Other:
- note added: "Last Updated: 16/11/2017, 00:22"
- note removed: "Last Updated: 16/11/2017, 00:04"
Changed lines of the file:
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@@
 <part name="GND8" library="SparkFun-Aesthetics" deviceset="GND" device=""/>
 <part name="FRAME1" library="frames" deviceset="A4L-LOC" device=""/>
+<part name="LOGO1" library="SparkFun-Aesthetics" deviceset="OSHW-LOGO" device="L"/>
 </parts>
 <sheets>
@@
 <text x="162.56" y="17.78" size="1.778" layer="94">18650 Battery Powered Temperature Sensors
 Based on MySensors Library with Arduino 3.3v</text>
-<text x="216.916" y="10.668" size="1.778" layer="94">Last Updated: 16/11/2017, 00:04</text>
+<text x="216.916" y="10.668" size="1.778" layer="94">Last Updated: 16/11/2017, 00:22</text>
 <text x="216.916" y="14.986" size="1.9304" layer="94">http://www.pihome.eu</text>
 </plain>
@@
 <attribute name="SHEET" x="230.505" y="5.08" size="2.54" layer="94"/>
 </instance>
+<instance part="LOGO1" gate="G$1" x="233.68" y="38.1"/>
 </instances>
 <busses>

Commit message: Improved PCB Design
Improved PCB Design
Parts:
- added LED1: (no value), adafruit:LED3MM
- added R5: 220Ohm, SparkFun-Resistors:RESISTORAXIAL-0.3
Connections:
- new net D4: R5.1, U$1.D4
- new net N$1: LED1.A, R5.2
- net GND: now also LED1.C
Changed lines of the file:
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@@
 <?xml version="1.0" encoding="utf-8"?>
 <!DOCTYPE eagle SYSTEM "eagle.dtd">
-<eagle version="7.5.0">
+<eagle version="9.0.1">
 <drawing>
 <settings>
 <setting alwaysvectorfont="no"/>
+<setting keepoldvectorfont="yes"/>
 <setting verticaltext="up"/>
 </settings>
@@
 <part name="FRAME1" library="frames" deviceset="A4L-LOC" device=""/>
 <part name="LOGO1" library="SparkFun-Aesthetics" deviceset="OSHW-LOGO" device="L"/>
+<part name="LED1" library="adafruit" deviceset="LED" device="3MM"/>
+<part name="GND12" library="SparkFun-Aesthetics" deviceset="GND" device=""/>
+<part name="R5" library="SparkFun-Resistors" deviceset="RESISTOR" device="AXIAL-0.3" value="220Ohm"/>
 </parts>
 <sheets>
@@
 </instance>
 <instance part="LOGO1" gate="G$1" x="233.68" y="38.1"/>
+<instance part="LED1" gate="G$1" x="93.98" y="58.42"/>
+<instance part="GND12" gate="1" x="93.98" y="48.26"/>
+<instance part="R5" gate="G$1" x="93.98" y="68.58" rot="R270"/>
 </instances>
 <busses>
@@
 <pinref part="GND8" gate="1" pin="GND"/>
 <wire x1="45.72" y1="104.14" x2="45.72" y2="114.3" width="0.1524" layer="91"/>
+</segment>
+<segment>
+<pinref part="GND12" gate="1" pin="GND"/>
+<pinref part="LED1" gate="G$1" pin="C"/>
+<wire x1="93.98" y1="53.34" x2="93.98" y2="50.8" width="0.1524" layer="91"/>
 </segment>
 </net>
@@
 </segment>
 </net>
+<net name="N$1" class="0">
+<segment>
+<pinref part="LED1" gate="G$1" pin="A"/>
+<pinref part="R5" gate="G$1" pin="2"/>
+<wire x1="93.98" y1="63.5" x2="93.98" y2="60.96" width="0.1524" layer="91"/>
+</segment>
+</net>
+<net name="D4" class="0">
+<segment>
+<pinref part="U$1" gate="G$1" pin="D4"/>
+<wire x1="22.86" y1="73.66" x2="17.78" y2="73.66" width="0.1524" layer="91"/>
+<label x="17.78" y="73.66" size="0.8128" layer="95" rot="R180" xref="yes"/>
+</segment>
+<segment>
+<pinref part="R5" gate="G$1" pin="1"/>
+<wire x1="93.98" y1="73.66" x2="93.98" y2="78.74" width="0.1524" layer="91"/>
+<label x="93.98" y="78.74" size="1.016" layer="95" rot="R90" xref="yes"/>
+</segment>
+</net>
